File: kicad/rp2350/lcdtap_rp2350.kicad_pcb (KiCad board)
At the start: 2 copper layers, 122 x 50 mm, 116 parts, among them J1 HDMI-001S, J2 Conn_02x08_Odd_Even, J3 Conn_01x03, J4 Conn_02x08_Odd_Even, J5 Conn_02x04_Odd_Even, P1 TYPE-C16PIN, SW1 SKRPACE010, SW2 SKRPACE010, SW3 SSSS811101, SW4 SKRPACE010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

Commit message: PCB artwork draft
Parts:
- moved C27 107.8 mm to (65.8, 125.5)
- moved R32 107.8 mm to (61.3, 146.4)
- moved C26 107.8 mm to (57.3, 129.9)
- moved C28 107.8 mm to (68.9, 125.0)
- moved D9 107.8 mm to (67.0, 151.2)
- moved H5 107.8 mm to (40.0, 112.0)
- moved H6 107.8 mm to (40.0, 152.0)
- moved H7 107.8 mm to (80.0, 112.0)
- moved H8 107.8 mm to (80.0, 152.0)
- moved J4 107.8 mm to (68.9, 112.7)
- moved J5 107.8 mm to (63.8, 149.3)
- moved R30 107.8 mm to (57.5, 146.4)
- moved U4 107.8 mm to (60.0, 122.5)
- moved U5 107.8 mm to (59.9, 139.7)
- moved U6 107.8 mm to (60.0, 131.0)
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Connections:
- SW3 pad 2: /SW_720P -> GND
Routing:
- net /SW_720P: track 60.8 -> 57.8 mm
- net Net-(J1-HPD): track 10.8 -> 11.3 mm
- net Net-(J1-UTILITY): track 18.9 -> 19.4 mm
- net Net-(J1-SDA): track 12.1 -> 12.6 mm
- net Net-(J1-SCL): track 17.5 -> 18.0 mm
- net Net-(J1-CEC): track 20.2 -> 20.7 mm
- net GND: vias 218 -> 219
Other:
- board size 122 x 50 mm -> 50 x 122 mm
- board text added: "-"
- board text added: "1V1"
- board text added: "3V3"
- board text added: "480P"
- board text added: "720P"
- board text added: "BOOT SEL"
- board text added: "CEC"
- board text added: "CS"
- board text added: "D+"
- board text added: "D-"
- board text added: "D0"
- board text added: "D1"
- board text added: "D2"
- board text added: "D3"
- board text added: "D4"
- board text added: "D5"
- board text added: "D6"
- board text added: "D7"
- board text added: "DC"
- board text added: "GND"
- board text added: "GPIO23"
- board text added: "GPIO24"
- board text added: "GPIO29"
- board text added: "HPD"
- board text added: "I2C/SPI Mode"
- board text added: "MOSI"
- board text added: "Parallel Mode"
- board text added: "RESET"
- board text added: "RST"
- board text added: "SCL"
- board text added: "SCLK"
- board text added: "SDA"
- board text added: "SWCLK"
- board text added: "SWDIO"
- board text added: "UTL"
- board text added: "VSYS"
- board text added: "WR"

Commit message: fix PCB
Parts:
- added D10: DF2B7AE, Diode_SMD:D_SOD-523, F.Cu at (59.3, 145.9)
- added D11: DF2B7AE, Diode_SMD:D_SOD-523, F.Cu at (63.1, 145.9)
- added D12: DF2B7AE, Diode_SMD:D_SOD-523, F.Cu at (54.4, 145.9)
- added G***: LOGO, LOGO, F.Cu at (43.8, 124.3)
- added G***: LOGO, LOGO, F.Cu at (42.4, 58.4)
- added G***: LOGO, LOGO, F.Cu at (40.5, 67.8)
- moved R4 0.21 mm to (49.1, 44.6)
- moved D3 0.20 mm to (51.0, 44.5), turned to -90 degrees
- moved D1 0.10 mm to (45.6, 46.3), turned to 180 degrees
- moved D2 0.10 mm to (48.4, 46.3), turned to 0 degrees
- turned D7 to 90 degrees
- turned D8 to -90 degrees
- turned D9 to 90 degrees
Connections:
- D1 pad 1: GND -> /USB_DP
- D1 pad 2: /USB_DP -> GND
- D2 pad 1: GND -> /USB_DM
- D2 pad 2: /USB_DM -> GND
- D3 pad 1: GND -> VBUS
- D3 pad 2: VBUS -> GND
- D7 pad 1: GND -> Net-(D7-A1)
- D7 pad 2: Net-(D7-A2) -> GND
- D8 pad 1: GND -> Net-(D8-A1)
- D8 pad 2: Net-(D8-A2) -> GND
- D9 pad 1: EXDES_GND -> EXDES_3V3
- D9 pad 2: EXDES_3V3 -> EXDES_GND
- J3 pad 1: Net-(D8-A2) -> Net-(D8-A1)
- J3 pad 3: Net-(D7-A2) -> Net-(D7-A1)
- J5 pad 2: Net-(J5-Pin_2) -> /EXDES_CS
- R16 pad 1: Net-(D8-A2) -> Net-(D8-A1)
- R17 pad 1: Net-(D7-A2) -> Net-(D7-A1)
- R31 pad 1: Net-(J5-Pin_2) -> /EXDES_CS
- R31 pad 2: /EXDES_CS -> Net-(D12-A1)
- U5 pad 11: /EXDES_CS -> Net-(D12-A1)
Routing:
- net Net-(D8-A2): track 31.0 -> 0.00 mm
- net Net-(D8-A1): track 0.00 -> 31.0 mm
- net Net-(D7-A2): track 26.0 -> 0.00 mm
- net Net-(D7-A1): track 0.00 -> 26.0 mm
- net Net-(D12-A1): track 0.00 -> 5.57 mm
- net Net-(J5-Pin_2): track 2.44 -> 0.00 mm
- net GND: track 27.4 -> 25.6 mm, vias 219 -> 221
- net VSYS: track 92.9 -> 94.1 mm
- net /EXDES_SCLK: track 34.8 -> 35.9 mm
- net /EXDES_CS: track 42.2 -> 43.0 mm
- net EXDES_GND: vias 102 -> 100
Other:
- board text added: "BOOTSEL"
- board text added: "Deserializer Addin"
- board text added: "Rev.1"
- board text added: "SPI/I2C Mode"
- board text removed: "BOOT SEL"
- board text removed: "I2C/SPI Mode"

Commit message: fix PCB
Parts:
- removed the G*** at (40.5, 67.8)
- added G***: LOGO, LOGO, B.Cu at (60.0, 131.0)
- added G***: LOGO, LOGO, B.Cu at (60.0, 77.0)
- added R34: 10k, Resistor_SMD:R_0402_1005Metric, F.Cu at (53.2, 45.3)
- added R35: 10k, Resistor_SMD:R_0402_1005Metric, F.Cu at (60.6, 127.2)
- added TP14: TestPoint_Small, TestPoint:TestPoint_Pad_D1.0mm, B.Cu at (53.2, 39.7)
- added TP15: TestPoint_Small, TestPoint:TestPoint_Pad_D1.0mm, F.Cu at (62.1, 127.5)
- added TP16: TestPoint_Small, TestPoint:TestPoint_Pad_D1.0mm, F.Cu at (58.0, 134.6)
- D1, D10, D11, D12, D2, D3, D7, D8, D9: value DF2B7AE -> SESD5Z5V
- moved C26 1.97 mm to (55.3, 130.2)
- moved U6 1.97 mm to (58.0, 131.3)
Connections:
- U3 pad 2: VSYS -> Net-(U3-EN)
- U4 pad 13: EXDES_GND -> Net-(U4-~{OE})
Routing:
- net Net-(U3-EN): track 0.00 -> 6.69 mm, vias 0 -> 1
- net Net-(U4-~{OE}): track 0.00 -> 3.57 mm
- net VSYS: track 94.1 -> 90.8 mm
- net EXDES_3V3: track 73.7 -> 75.8 mm
- net EXDES_GND: track 1.74 -> 0.00 mm
- net Net-(U5-QC): track 5.92 -> 4.85 mm
- net /EXDES_MOSI: track 34.4 -> 33.8 mm
- net GND: vias 221 -> 220
Other:
- board text added: "3V3_EN"
- board text added: "Deserializer Addin Rev.1"
- board text removed: "Deserializer Addin"

Commit message: fix PCB
Parts:
- removed D7, D8: SESD5Z5V, Diode_SMD:D_SOD-523
- moved J3 18.7 mm to (82.5, 68.8)
- moved R16 6.55 mm to (79.7, 66.8), turned to 180 degrees
- moved R17 5.20 mm to (79.7, 65.8), turned to 180 degrees
- moved TP10 4.10 mm to (73.0, 72.1)
Routing:
- net Net-(J3-Pin_1): track 31.0 -> 3.15 mm
- net Net-(J3-Pin_3): track 26.0 -> 3.12 mm
- net Net-(U1-SWCLK): track 15.2 -> 23.4 mm
- net Net-(U1-SWDIO): track 16.2 -> 23.6 mm
- net Net-(U1-RUN): track 34.8 -> 35.6 mm
- net GND: vias 220 -> 216
Other:
- board text added: "BOOT SEL"
- board text removed: "BOOTSEL"

Commit message: fix PCB
Connections:
- net Net-(U1-VREG_AVDD) renamed VREG_AVDD
Changed lines of the file:
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@@
 			(layers "F.Cu" "F.Mask" "F.Paste")
 			(roundrect_rratio 0.25)
-			(net "Net-(U1-VREG_AVDD)")
+			(net "VREG_AVDD")
 			(pintype "passive")
 		)
@@
 			(layers "F.Cu" "F.Mask" "F.Paste")
 			(roundrect_rratio 0.25)
-			(net "Net-(U1-VREG_AVDD)")
+			(net "VREG_AVDD")
 			(pintype "passive")
 		)
@@
 			(layers "F.Cu" "F.Mask" "F.Paste")
 			(roundrect_rratio 0.25)
-			(net "Net-(U1-VREG_AVDD)")
+			(net "VREG_AVDD")
 			(pinfunction "VREG_AVDD_46")
 			(pintype "power_in")
@@
 	)
 	(segment
-		(start 53.5 55.1)
-		(end 54.45 55.1)
-		(width 0.2)
-		(layer "F.Cu")
-		(net "Net-(U1-VREG_AVDD)")
-	)
-	(segment
-		(start 56.55 56.9)
-		(end 56.55 56.95)
-		(width 0.2)
-		(layer "F.Cu")
-		(net "Net-(U1-VREG_AVDD)")
-	)
-	(segment
-		(start 54.75 55.1)
-		(end 56.55 56.9)
-		(width 0.2)
-		(layer "F.Cu")
-		(net "Net-(U1-VREG_AVDD)")
-	)
-	(segment
-		(start 53.2 54.8)
-		(end 53.5 55.1)
-		(width 0.2)
-		(layer "F.Cu")
-		(net "Net-(U1-VREG_AVDD)")
-	)
-	(segment
-		(start 54.7 55.1)
-		(end 54.75 55.1)
-		(width 0.2)
-		(layer "F.Cu")
-		(net "Net-(U1-VREG_AVDD)")
-	)
-	(segment
-		(start 56.55 56.95)
-		(end 56.55 57.2)
-		(width 0.2)
-		(layer "F.Cu")
-		(net "Net-(U1-VREG_AVDD)")
-	)
-	(segment
-		(start 54.45 55.1)
-		(end 54.7 55.1)
-		(width 0.15)
-		(layer "F.Cu")
-		(net "Net-(U1-VREG_AVDD)")
-	)
-	(segment
 		(start 59.9 69.2)
 		(end 59.4 69.7)
@@
 		(net "Net-(U1-GPIO29{slash}ADC3)")
 	)
+	(segment
+		(start 53.5 55.1)
+		(end 54.45 55.1)
+		(width 0.2)
+		(layer "F.Cu")
+		(net "VREG_AVDD")
+	)
+	(segment
+		(start 56.55 56.9)
+		(end 56.55 56.95)
+		(width 0.2)
+		(layer "F.Cu")
+		(net "VREG_AVDD")
+	)
+	(segment
+		(start 54.75 55.1)
+		(end 56.55 56.9)
+		(width 0.2)
+		(layer "F.Cu")
+		(net "VREG_AVDD")
+	)
+	(segment
+		(start 53.2 54.8)
+		(end 53.5 55.1)
+		(width 0.2)
+		(layer "F.Cu")
+		(net "VREG_AVDD")
+	)
+	(segment
+		(start 54.7 55.1)
+		(end 54.75 55.1)
+		(width 0.2)
+		(layer "F.Cu")
+		(net "VREG_AVDD")
+	)
+	(segment
+		(start 56.55 56.95)
+		(end 56.55 57.2)
+		(width 0.2)
+		(layer "F.Cu")
+		(net "VREG_AVDD")
+	)
+	(segment
+		(start 54.45 55.1)
+		(end 54.7 55.1)
+		(width 0.15)
+		(layer "F.Cu")
+		(net "VREG_AVDD")
+	)
 	(zone
