File: kicad/rp2350/lcdtap_rp2350.kicad_pcb (KiCad board)
At the start: 2 copper layers, 50 x 122 mm, 126 parts, among them J1 HDMI-001S, J2 Conn_02x08_Odd_Even, J3 Conn_01x03, J4 Conn_02x08_Odd_Even, J5 Conn_02x04_Odd_Even, P1 TYPE-C16PIN, SW1 SKRPACE010, SW2 SKRPACE010, SW3 SSSS811101, SW4 SKRPACE010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

Commit message: PCB rev.2
Parts:
- added JP2: SolderJumper_2_Open_Small, Jumper:SolderJumper-2_P1.3mm_Open_RoundedPad1.0x1.5mm, B.Cu at (67.7, 39.4)
Connections:
- J1 pad 18: VBUS -> VIDEO_5V
Routing:
- net VBUS: track 45.3 -> 34.1 mm, vias 4 -> 5
- net VIDEO_5V: track 0.00 -> 9.90 mm, vias 0 -> 1
Other:
- board text added: "Rev.2"
- board text removed: "Rev.1"
