File: kicad/rp2350/lcdtap_rp2350.kicad_sch (KiCad schematic)
At the start: 112 parts, among them J1 HDMI-001S, J2 Conn_02x08_Odd_Even, J3 Conn_01x03, J4 Conn_02x08_Odd_Even, J5 Conn_02x04_Odd_Even, P1 TYPE-C16PIN, SW1 SKRPACE010, SW2 SKRPACE010, SW3 SSSS811101, SW4 SKRPACE010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

Commit message: PCB artwork draft
Parts:
- added C28: 10u, Capacitor_SMD:C_0603_1608Metric, symbol Device:C_Small
- added R33: 33, Resistor_SMD:R_0402_1005Metric, symbol Device:R_Small
- C1, C2: value 10u -> 4.7u; LCSC C19702 -> C19666
- J1: footprint Connector_Video:HDMI_A_Molex_208658-1001_Horizontal -> shpc_mechanical:HDMI_A_Molex_208658-1001_Horizontal_Edge
- J2: footprint Connector_PinHeader_2.54mm:PinHeader_2x08_P2.54mm_Horizontal -> shpc_mechanical:PinHeader_2x08_P2.54mm_Horizontal_Rev
- J4: footprint Connector_PinSocket_2.54mm:PinSocket_2x08_P2.54mm_Horizontal -> shpc_mechanical:PinSocket_2x08_P2.54mm_Horizontal_Rev
- J5: footprint Connector_PinHeader_2.54mm:PinHeader_2x04_P2.54mm_Horizontal -> shpc_mechanical:PinHeader_2x04_P2.54mm_Horizontal_Rev
- L1: value LQM31PN3R3M00L -> AOTA-B201610S3R3-101-T; footprint Inductor_SMD:L_1206_3216Metric -> shpc_discreet:AOTA-B201610S3R3-101-T; symbol Device:L_Small -> shpc_discreet:Inductor_with_mark; LCSC C91612 -> C42411119
- TP1, TP10, TP11, TP12, TP13, TP2, TP3, TP4, TP5, TP6, TP7, TP8, TP9: footprint TestPoint:TestPoint_Pad_D2.0mm -> TestPoint:TestPoint_Pad_D1.0mm
- Y1: value X322512MSB4SI -> ABM8-272-T3; LCSC C9002 -> C20625731
Connections:
- net 3V3: now also R33.1; no longer C16.1, U1.46 (VREG_AVDD)
- net EXDES_3V3: now also C28.1
- net EXDES_GND: now also D9.1 (A1), C28.2
- net GND: now also SW3.SH; no longer D9.1 (A1), SW3. (SH)
- net KEY_RIGHT: now reaches SW5.2, U1.41 (GPIO27/ADC1)
- net KEY_DOWN: now reaches SW8.2, U1.33 (GPIO21)
- net SW_720P: now reaches SW3.1 (A), SW3.2 (B), U1.32 (GPIO20)
- net KEY_LEFT: now reaches SW7.2, U1.34 (GPIO22)
- net at U1.35 (GPIO23): now also TP6.1; no longer R15.1
- net at U1.36 (GPIO24): now also TP7.1; no longer TP6.1
- net LED: now reaches U1.37 (GPIO25)
- net LED: now also R15.1; no longer TP7.1
- net KEY_UP: now reaches SW6.2, U1.40 (GPIO26/ADC0)
- net KEY_ENTER: now reaches SW4.2, U1.42 (GPIO28/ADC2)
- new net: C16.1, R33.2, U1.46 (VREG_AVDD)
Other:
- moved on the sheet: D9

Commit message: PCB artwork draft
Connections:
- net GND: now also SW3.2 (B)
- net SW_720P: no longer SW3.2 (B)
Other:
- moved on the sheet: SW3
Changed lines of the file:
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@@
 	)
 	(junction
-		(at 307.34 123.19)
-		(diameter 0)
-		(color 0 0 0 0)
-	)
-	(junction
 		(at 124.46 78.74)
 		(diameter 0)
@@
 	(wire
 		(pts
-			(xy 307.34 129.54) (xy 308.61 129.54)
-		)
-		(stroke
-			(width 0)
-			(type default)
-		)
-	)
-	(wire
-		(pts
 			(xy 85.09 40.64) (xy 85.09 38.1)
 		)
@@
 	(wire
 		(pts
-			(xy 320.04 127) (xy 320.04 123.19)
-		)
-		(stroke
-			(width 0)
-			(type default)
-		)
-	)
-	(wire
-		(pts
 			(xy 246.38 200.66) (xy 259.08 200.66)
 		)
@@
 	(wire
 		(pts
-			(xy 318.77 127) (xy 320.04 127)
+			(xy 312.42 127) (xy 311.15 127)
 		)
 		(stroke
@@
 	(wire
 		(pts
-			(xy 307.34 123.19) (xy 307.34 129.54)
+			(xy 311.15 104.14) (xy 311.15 127)
 		)
 		(stroke
@@
 	(wire
 		(pts
+			(xy 323.85 129.54) (xy 323.85 137.16)
+		)
+		(stroke
+			(width 0)
+			(type default)
+		)
+	)
+	(wire
+		(pts
 			(xy 74.93 43.18) (xy 95.25 43.18)
 		)
@@
 	(wire
 		(pts
-			(xy 318.77 132.08) (xy 320.04 132.08)
+			(xy 312.42 132.08) (xy 311.15 132.08)
 		)
 		(stroke
@@
 	(wire
 		(pts
-			(xy 320.04 123.19) (xy 307.34 123.19)
-		)
-		(stroke
-			(width 0)
-			(type default)
-		)
-	)
-	(wire
-		(pts
 			(xy 152.4 38.1) (xy 154.94 38.1)
 		)
@@
 	(wire
 		(pts
-			(xy 320.04 137.16) (xy 320.04 132.08)
+			(xy 311.15 137.16) (xy 311.15 132.08)
 		)
 		(stroke
@@
 	(wire
 		(pts
+			(xy 323.85 129.54) (xy 322.58 129.54)
+		)
+		(stroke
+			(width 0)
+			(type default)
+		)
+	)
+	(wire
+		(pts
 			(xy 50.8 83.82) (xy 53.34 83.82)
 		)
@@
 	(wire
 		(pts
-			(xy 313.69 135.89) (xy 313.69 137.16)
+			(xy 317.5 135.89) (xy 317.5 137.16)
 		)
 		(stroke
@@
 	(wire
 		(pts
-			(xy 254 104.14) (xy 307.34 104.14)
+			(xy 254 104.14) (xy 311.15 104.14)
 		)
 		(stroke
@@
 	(wire
 		(pts
-			(xy 307.34 104.14) (xy 307.34 123.19)
-		)
-		(stroke
-			(width 0)
-			(type default)
-		)
-	)
-	(wire
-		(pts
 			(xy 35.56 106.68) (xy 35.56 110.49)
 		)
@@
 	(symbol
 		(lib_id "power:GND")
-		(at 320.04 137.16 0)
+		(at 311.15 137.16 0)
+		(mirror y)
 		(unit 1)
 		(body_style 1)
@@
 		(fields_autoplaced yes)
 		(property "Reference" "#PWR051"
-			(at 320.04 143.51 0)
+			(at 311.15 143.51 0)
 			(hide yes)
 			(show_name no)
@@
 		)
 		(property "Value" "GND"
-			(at 320.04 142.24 0)
+			(at 311.15 142.24 0)
 			(show_name no)
 			(do_not_autoplace no)
@@
 		)
 		(property "Footprint" ""
-			(at 320.04 137.16 0)
+			(at 311.15 137.16 0)
 			(hide yes)
 			(show_name no)
@@
 		)
 		(property "Datasheet" ""
-			(at 320.04 137.16 0)
+			(at 311.15 137.16 0)
 			(hide yes)
 			(show_name no)
@@
 		)
 		(property "Description" "Power symbol creates a global label with name \"GND\" , ground"
-			(at 320.04 137.16 0)
+			(at 311.15 137.16 0)
 			(hide yes)
 			(show_name no)
@@
 	)
 	(symbol
+		(lib_id "power:GND")
+		(at 323.85 137.16 0)
+		(mirror y)
+		(unit 1)
+		(body_style 1)
+		(exclude_from_sim no)
+		(in_bom yes)
+		(on_board yes)
+		(in_pos_files yes)
+		(dnp no)
+		(fields_autoplaced yes)
+		(property "Reference" "#PWR089"
+			(at 323.85 143.51 0)
+			(hide yes)
+			(show_name no)
+			(do_not_autoplace no)
+			(effects
+				(font
+					(size 1.27 1.27)
+				)
+			)
+		)
+		(property "Value" "GND"
+			(at 323.85 142.24 0)
+			(show_name no)
+			(do_not_autoplace no)
+			(effects
+				(font
+					(size 1.27 1.27)
+				)
+			)
+		)
+		(property "Footprint" ""
+			(at 323.85 137.16 0)
+			(hide yes)
+			(show_name no)
+			(do_not_autoplace no)
+			(effects
+				(font
+					(size 1.27 1.27)
+				)
+			)
+		)
+		(property "Datasheet" ""
+			(at 323.85 137.16 0)
+			(hide yes)
+			(show_name no)
+			(do_not_autoplace no)
+			(effects
+				(font
+					(size 1.27 1.27)
+				)
+			)
+		)
+		(property "Description" "Power symbol creates a global label with name \"GND\" , ground"
+			(at 323.85 137.16 0)
+			(hide yes)
+			(show_name no)
+			(do_not_autoplace no)
+			(effects
+				(font
+					(size 1.27 1.27)
+				)
+			)
+		)
+		(pin "1"
+		)
+		(instances
+			(project "lcdtap_rp2350"
+				(path "/bb6d9c56-6581-49df-a688-e642dbd096a3"
+					(reference "#PWR089")
+					(unit 1)
+				)
+			)
+		)
+	)
+	(symbol
 		(lib_id "Device:C_Small")
 		(at 105.41 43.18 0)
@@
 	(symbol
 		(lib_id "shpc_mechanical:SSSS811101")
-		(at 313.69 129.54 0)
+		(at 317.5 129.54 0)
+		(mirror y)
 		(unit 1)
 		(body_style 1)
@@
 		(dnp no)
 		(property "Reference" "SW3"
-			(at 308.61 119.38 0)
+			(at 311.912 121.158 0)
 			(show_name no)
 			(do_not_autoplace no)
@@
 					(size 1.27 1.27)
 				)
-				(justify left)
+				(justify right)
 			)
 		)
 		(property "Value" "SSSS811101"
-			(at 308.61 121.412 0)
+			(at 311.912 123.19 0)
 			(show_name no)
 			(do_not_autoplace no)
@@
 					(size 1.27 1.27)
 				)
-				(justify left)
+				(justify right)
 			)
 		)
 		(property "Footprint" "shpc_mechanical:SW_SPDT_Alps_SSSS811101"
-			(at 313.69 129.54 0)
+			(at 317.5 129.54 0)
 			(hide yes)
 			(show_name no)
@@
 		)
 		(property "Datasheet" "https://jlc-prod-smt.oss-eu-central-1.aliyuncs.com/smtDataManualFile/8588894528888066048-C109335.pdf"
-			(at 313.69 137.16 0)
+			(at 317.5 137.16 0)
 			(hide yes)
 			(show_name no)
@@
 		)
 		(property "Description" "Switch, single pole double throw"
-			(at 313.69 129.54 0)
+			(at 317.5 129.54 0)
 			(hide yes)
 			(show_name no)
@@
 		)
 		(property "LCSC" "C109335"
-			(at 313.69 129.54 0)
+			(at 317.5 129.54 0)
 			(hide yes)
 			(show_name no)
@@
 	(symbol
 		(lib_id "power:GND")
-		(at 313.69 137.16 0)
+		(at 317.5 137.16 0)
+		(mirror y)
 		(unit 1)
 		(body_style 1)
@@
 		(fields_autoplaced yes)
 		(property "Reference" "#PWR049"
-			(at 313.69 143.51 0)
+			(at 317.5 143.51 0)
 			(hide yes)
 			(show_name no)
@@
 		)
 		(property "Value" "GND"
-			(at 313.69 142.24 0)
+			(at 317.5 142.24 0)
 			(show_name no)
 			(do_not_autoplace no)
@@
 		)
 		(property "Footprint" ""
-			(at 313.69 137.16 0)
+			(at 317.5 137.16 0)
 			(hide yes)
 			(show_name no)
@@
 		)
 		(property "Datasheet" ""
-			(at 313.69 137.16 0)
+			(at 317.5 137.16 0)
 			(hide yes)
 			(show_name no)
@@
 		)
 		(property "Description" "Power symbol creates a global label with name \"GND\" , ground"
-			(at 313.69 137.16 0)
+			(at 317.5 137.16 0)
 			(hide yes)
 			(show_name no)

Commit message: fix PCB
Parts:
- added D10, D11, D12: DF2B7AE, Diode_SMD:D_SOD-523, symbol Device:D_TVS_Small
- J2, J4, J5: now not fitted
Connections:
- net EXDES_3V3: now also D9.1 (A1); no longer D9.2 (A2)
- net EXDES_CS: now also J5.2 (Pin_2), R31.1; no longer R31.2, U5.11 (CLR)
- net EXDES_GND: now also D9.2 (A2), D10.2 (A2), D11.2 (A2), D12.2 (A2); no longer D9.1 (A1)
- net EXDES_MOSI: now also D11.1 (A1)
- net EXDES_SCLK: now also D10.1 (A1)
- net GND: now also D1.2 (A2), D2.2 (A2), D3.2 (A2), D7.2 (A2), D8.2 (A2); no longer D1.1 (A1), D2.1 (A1), D3.1 (A1), D7.1 (A1), D8.1 (A1)
- net USB_DM: now also D2.1 (A1); no longer D2.2 (A2)
- net USB_DP: now also D1.1 (A1); no longer D1.2 (A2)
- net VBUS: now also D3.1 (A1); no longer D3.2 (A2)
- net at J3.1 (Pin_1), R16.1: now also D8.1 (A1); no longer D8.2 (A2)
- net at J3.3 (Pin_3), R17.1: now also D7.1 (A1); no longer D7.2 (A2)
- new net: D12.1 (A1), R31.2, U5.11 (CLR)
Other:
- moved on the sheet: C25, C26, C27, D3, R30, R32, U4, U5, U6

Commit message: fix PCB
Parts:
- added R34, R35: 10k, Resistor_SMD:R_0402_1005Metric, symbol Device:R_Small
- added TP14, TP15, TP16: TestPoint_Small, TestPoint:TestPoint_Pad_D1.0mm, symbol Connector:TestPoint_Small
- D1, D10, D11, D12, D2, D3, D7, D8, D9: value DF2B7AE -> SESD5Z5V; LCSC C1973289 -> C19631222
- J2: LCSC C2894988 -> (none); now left out of the parts list
- J3, TP1, TP10, TP11, TP12, TP13, TP2, TP3, TP4, TP5, TP6, TP7, TP8, TP9: now left out of the parts list
- J4: LCSC C2897428 -> (none); now left out of the parts list
- J5: LCSC C492432 -> (none); now left out of the parts list
- U4: LCSC (none) -> C5947
- U5: LCSC C6848 -> C27387
Connections:
- net EXDES_GND: now also R35.1; no longer U4.13 (~{OE})
- net VSYS: now also R34.1; no longer U3.2 (EN)
- net at U5.6 (QC), U6.2: now also TP16.1
- new net: R35.2, TP15.1, U4.13 (~{OE})
- new net: R34.2, TP14.1, U3.2 (EN)
Other:
- moved on the sheet: C19, C20, C21, C22, C23, C24, C25, C26, D12, D5, L2, R31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

Commit message: fix PCB
Parts:
- removed D7, D8: SESD5Z5V, Diode_SMD:D_SOD-523, symbol Device:D_TVS_Small
Other:
- moved on the sheet: J3

Commit message: fix PCB
Connections:
- net VREG_AVDD: now reaches C16.1, R33.2, U1.46 (VREG_AVDD)

Commit message: PCB rev.2
Parts:
- added JP2: SolderJumper_2_Open_Small, Jumper:SolderJumper-2_P1.3mm_Open_RoundedPad1.0x1.5mm, symbol shpc_mechanical:SolderJumper_2_Open_Small
Connections:
- net VBUS: now also JP2.1 (A); no longer J1.18 (+5V)
- new net VIDEO_5V: J1.18 (+5V), JP2.2 (B)
Other:
- moved on the sheet: J1, TP1, TP2, TP3, TP4, TP5
