File: example/pico2_universal/kicad/lcdtap_rp2350.kicad_pcb (KiCad board)
At the start: 2 copper layers, 50 x 122 mm, 127 parts, among them J1 HDMI-001S, J2 Conn_02x08_Odd_Even, J3 Conn_01x03, J4 Conn_02x08_Odd_Even, J5 Conn_02x04_Odd_Even, P1 TYPE-C16PIN, SW1 SKRPACE010, SW2 SKRPACE010, SW3 SSSS811101, SW4 SKRPACE010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

Commit message: fix PCB
Parts:
- removed C25, C26, C27: 100n, Capacitor_SMD:C_0402_1005Metric
- removed C28: 10u, Capacitor_SMD:C_0603_1608Metric
- removed D10, D11, D12, D9: SESD5Z5V, Diode_SMD:D_SOD-523
- removed the G*** at (43.8, 124.3)
- removed the G*** at (60.0, 131.0)
- removed H5, H6, H7, H8: MountingHole, MountingHole:MountingHole_3.5mm
- removed J4: Conn_02x08_Odd_Even, shpc_mechanical:PinSocket_2x08_P2.54mm_Horizontal_Rev
- removed J5: Conn_02x04_Odd_Even, shpc_mechanical:PinHeader_2x04_P2.54mm_Horizontal_Rev
- removed R30, R31, R32: 47, Resistor_SMD:R_0402_1005Metric
- removed R35: 10k, Resistor_SMD:R_0402_1005Metric
- removed REF** (x2): JLC_MouseBites, shpc_mechanical:JLC_MouseBites
- removed TP15, TP16: TestPoint_Small, TestPoint:TestPoint_Pad_D1.0mm
- removed U4: 74HC595, Package_SO:SOIC-16_3.9x9.9mm_P1.27mm
- removed U5: 74HC4040, Package_SO:SOIC-16_3.9x9.9mm_P1.27mm
- removed U6: 74LVC1G04, Package_TO_SOT_SMD:SOT-23-5
Routing:
- net EXDES_3V3: track 75.8 -> 0.00 mm, vias 4 -> 0
- net /EXDES_DC: track 54.1 -> 0.00 mm
- net /EXDES_RST: track 49.7 -> 0.00 mm
- net /EXDES_CS: track 43.0 -> 0.00 mm
- net /EXDES_SCLK: track 35.9 -> 0.00 mm
- net /EXDES_MOSI: track 33.8 -> 0.00 mm
- net /EXDES_WR: track 26.2 -> 0.00 mm
- net /EXDES_D6: track 25.7 -> 0.00 mm
- net /EXDES_D7: track 22.8 -> 0.00 mm
- net /EXDES_D5: track 22.7 -> 0.00 mm
- net /EXDES_D0: track 22.6 -> 0.00 mm
- net /EXDES_D4: track 15.7 -> 0.00 mm
- net /EXDES_D3: track 14.4 -> 0.00 mm
- net /EXDES_D1: track 14.3 -> 0.00 mm
- net /EXDES_D2: track 9.84 -> 0.00 mm
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- removed copper zone on B.Cu, net EXDES_GND
- removed copper zone on F.Cu, net EXDES_GND
Other:
- board size 50 x 122 mm -> 50 x 70 mm
- board text added: "5V_VIDEO"
- board text removed: "Deserializer Addin Rev.1"
