File: example/pico2_universal/kicad/lcdtap_rp2350.kicad_sch (KiCad schematic)
At the start: 121 parts, among them J1 HDMI-001S, J2 Conn_02x08_Odd_Even, J3 Conn_01x03, J4 Conn_02x08_Odd_Even, J5 Conn_02x04_Odd_Even, P1 TYPE-C16PIN, SW1 SKRPACE010, SW2 SKRPACE010, SW3 SSSS811101, SW4 SKRPACE010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

Commit message: fix PCB
Parts:
- removed C25, C26, C27: 100n, Capacitor_SMD:C_0402_1005Metric, symbol Device:C_Small
- removed C28: 10u, Capacitor_SMD:C_0603_1608Metric, symbol Device:C_Small
- removed D10, D11, D12, D9: SESD5Z5V, Diode_SMD:D_SOD-523, symbol Device:D_TVS_Small
- removed H5, H6, H7, H8: MountingHole, MountingHole:MountingHole_3.5mm, symbol Mechanical:MountingHole
- removed J4: Conn_02x08_Odd_Even, shpc_mechanical:PinSocket_2x08_P2.54mm_Horizontal_Rev, symbol Connector_Generic:Conn_02x08_Odd_Even
- removed J5: Conn_02x04_Odd_Even, shpc_mechanical:PinHeader_2x04_P2.54mm_Horizontal_Rev, symbol Connector_Generic:Conn_02x04_Odd_Even
- removed R30, R31, R32: 47, Resistor_SMD:R_0402_1005Metric, symbol Device:R_Small
- removed R35: 10k, Resistor_SMD:R_0402_1005Metric, symbol Device:R_Small
- removed TP15, TP16: TestPoint_Small, TestPoint:TestPoint_Pad_D1.0mm, symbol Connector:TestPoint_Small
- removed U4: 74HC595, Package_SO:SOIC-16_3.9x9.9mm_P1.27mm, symbol 74xx:74HC595
- removed U5: 74HC4040, Package_SO:SOIC-16_3.9x9.9mm_P1.27mm, symbol shpc_ic:74HC4040
- removed U6: 74LVC1G04, Package_TO_SOT_SMD:SOT-23-5, symbol 74xGxx:74LVC1G04
Connections:
- no-connect marks 16 -> 2
